File: Kicad/Kicad.kicad_pcb (KiCad board)
At the start: 2 copper layers, 65.3 x 57 mm, 24 parts, among them J1 Conn_01x04_Male, J2 Conn_01x04_Male, J3 Conn_01x03_Male, J4 Conn_01x04_Male, J5 Conn_01x03_Male, J6 Conn_01x03_Male, J7 Conn_01x02_Female, J8 Conn_01x02_Female, J9 Conn_01x02_Female, P1 Conn_02x20_Odd_Even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

Commit message: Modification Kicad
Parts:
- moved J2 6.88 mm to (242.6, 113.6)
- moved R2 5.21 mm to (232.4, 109.2)
Routing:
- net /GPIO11(SPI0_SCK): track 33.0 -> 48.8 mm, vias 0 -> 1
- net +3V3: track 71.9 -> 59.0 mm, vias 0 -> 1
- net /GPIO5: track 50.4 -> 58.6 mm, vias 0 -> 1
- net /GPIO8(SPI0_CE_N): track 62.9 -> 70.3 mm, vias 0 -> 1
- net /GPIO4(GCLK): track 27.4 -> 34.4 mm, vias 0 -> 1
- net /GPIO6: track 47.1 -> 52.1 mm, vias 0 -> 1
- net +5V: track 114.5 -> 116.8 mm, vias 0 -> 1
- net /GPIO9(SPI0_MISO): track 30.7 -> 31.6 mm, vias 0 -> 1
- net /GPIO27(GEN2): track 20.0 -> 20.4 mm, vias 0 -> 1
- net /GPIO22(GEN3): track 35.4 -> 35.5 mm, vias 0 -> 1
- net /GPIO10(SPI0_MOSI): vias 0 -> 1
